File: pcb/Numpad Keyboard/Numpad.kicad_sch (KiCad schematic)
At the start: 65 parts, among them J1 Conn_01x04, J2 Conn_01x04, U1 MAX7301ATL+, U2 IS31FL3743-QF, U3 IS31FL3743-QF

Commit message: Modified footprint for LEDs, so they have right rotation for pick and place
Parts:
- R2, R3: value R -> R 10 kOhm; symbol vakeyboard:R -> vakeyboard:R 10 kOhm
- U2, U3: Description / Value 10MHz 16 POR SPI SOIC-28_300mil I/O Expanders ROHS -> UQFN-40(5x5) LED Drivers ROHS; LCSC C47023 -> C2678953; Manufacturer Microchip Tech -> Lumissil Microsystems; Mfg Part # MCP23S17T-E/SO -> IS31FL3743A-QULS4-TR; Package/Footprint SOIC-28_7.5x17.9x1.27P -> QFN-40
Changed lines of the file:
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@@
     (pin "4")
   )
-  (symbol (lib_id "vakeyboard:R") (at 148.59 241.3 270) (unit 1)
+  (symbol (lib_id "vakeyboard:R 10 kOhm") (at 148.59 241.3 270) (unit 1)
     (in_bom yes) (on_board yes) (fields_autoplaced)
     (property "Reference" "R3" (id 0) (at 148.59 238.125 90))
-    (property "Value" "R" (id 1) (at 148.59 241.3 90)
-      (effects (font (size 1.27 1.27)) hide)
-    )
-    (property "Footprint" "Footprints:R_0402_1005Metric" (id 2) (at 148.59 239.522 90)
-      (effects (font (size 1.27 1.27)) hide)
-    )
-    (property "Datasheet" "https://datasheet.lcsc.com/lcsc/2206010100_UNI-ROYAL-Uniroyal-Elec-0402WGF1002TCE_C25744.pdf" (id 3) (at 148.59 241.3 0)
-      (effects (font (size 1.27 1.27)) hide)
-    )
-    (property "Description / Value" "1/16W Thick Film Resistors 50V ±1% ±100ppm/℃ -55℃~+155℃ 10kΩ 0402  Chip Resistor - Surface Mount ROHS" (id 4) (at 148.59 241.3 0)
-      (effects (font (size 1.27 1.27)) hide)
-    )
-    (property "LCSC" "C25744" (id 5) (at 148.59 241.3 0)
-      (effects (font (size 1.27 1.27)) hide)
-    )
-    (property "Manufacturer" "UNI-ROYAL(Uniroyal Elec)" (id 6) (at 148.59 241.3 0)
-      (effects (font (size 1.27 1.27)) hide)
-    )
-    (property "Mfg Part #" "0402WGF1002TCE" (id 7) (at 148.59 241.3 0)
-      (effects (font (size 1.27 1.27)) hide)
-    )
-    (property "Package/Footprint" "0402" (id 8) (at 148.59 241.3 0)
-      (effects (font (size 1.27 1.27)) hide)
-    )
-    (property "Type" "SMD" (id 9) (at 148.59 241.3 0)
+    (property "Value" "R 10 kOhm" (id 1) (at 148.59 241.3 90)
+      (effects (font (size 1.27 1.27)) hide)
+    )
+    (property "Footprint" "Footprints:R_0402_1005Metric" (id 2) (at 114.3 240.03 0)
+      (effects (font (size 1.27 1.27)) hide)
+    )
+    (property "Datasheet" "https://datasheet.lcsc.com/lcsc/2206010100_UNI-ROYAL-Uniroyal-Elec-0402WGF1002TCE_C25744.pdf" (id 3) (at 132.08 242.57 0)
+      (effects (font (size 1.27 1.27)) hide)
+    )
+    (property "Description / Value" "1/16W Thick Film Resistors 50V ±1% ±100ppm/℃ -55℃~+155℃ 10kΩ 0402  Chip Resistor - Surface Mount ROHS" (id 4) (at 124.46 242.57 0)
+      (effects (font (size 1.27 1.27)) hide)
+    )
+    (property "LCSC" "C25744" (id 5) (at 121.92 241.3 0)
+      (effects (font (size 1.27 1.27)) hide)
+    )
+    (property "Manufacturer" "UNI-ROYAL(Uniroyal Elec)" (id 6) (at 129.54 242.57 0)
+      (effects (font (size 1.27 1.27)) hide)
+    )
+    (property "Mfg Part #" "0402WGF1002TCE" (id 7) (at 127 242.57 0)
+      (effects (font (size 1.27 1.27)) hide)
+    )
+    (property "Package/Footprint" "0402" (id 8) (at 119.38 241.3 0)
+      (effects (font (size 1.27 1.27)) hide)
+    )
+    (property "Type" "SMD" (id 9) (at 116.84 241.3 0)
       (effects (font (size 1.27 1.27)) hide)
     )
@@
     (pin "2")
   )
-  (symbol (lib_id "vakeyboard:IS31FL3743-QF") (at 59.055 219.71 90) (unit 1)
+  (symbol (lib_name "IS31FL3743-QF_1") (lib_id "vakeyboard:IS31FL3743-QF") (at 59.055 219.71 90) (unit 1)
     (in_bom yes) (on_board yes) (fields_autoplaced)
     (property "Reference" "U2" (id 0) (at 100.33 214.5155 90))
@@
       (effects (font (size 1.27 1.27)) hide)
     )
-    (property "Datasheet" "http://ww1.microchip.com/downloads/en/DeviceDoc/20001952C.pdf" (id 3) (at 59.055 219.71 0)
-      (effects (font (size 1.27 1.27)) hide)
-    )
-    (property "Description / Value" "10MHz 16 POR SPI SOIC-28_300mil  I/O Expanders ROHS" (id 4) (at 59.055 219.71 0)
-      (effects (font (size 1.27 1.27)) hide)
-    )
-    (property "LCSC" "C47023" (id 5) (at 59.055 219.71 0)
-      (effects (font (size 1.27 1.27)) hide)
-    )
-    (property "Manufacturer" "Microchip Tech" (id 6) (at 59.055 219.71 0)
-      (effects (font (size 1.27 1.27)) hide)
-    )
-    (property "Mfg Part #" "MCP23S17T-E/SO" (id 7) (at 59.055 219.71 0)
-      (effects (font (size 1.27 1.27)) hide)
-    )
-    (property "Package/Footprint" "SOIC-28_7.5x17.9x1.27P" (id 8) (at 59.055 219.71 0)
+    (property "Datasheet" "https://datasheet.lcsc.com/lcsc/2106070633_Lumissil-Microsystems-IS31FL3743A-QULS4-TR_C2678953.pdf" (id 3) (at 59.055 219.71 0)
+      (effects (font (size 1.27 1.27)) hide)
+    )
+    (property "Description / Value" "UQFN-40(5x5)  LED Drivers ROHS" (id 4) (at 59.055 219.71 0)
+      (effects (font (size 1.27 1.27)) hide)
+    )
+    (property "LCSC" "C2678953" (id 5) (at 59.055 219.71 0)
+      (effects (font (size 1.27 1.27)) hide)
+    )
+    (property "Manufacturer" "Lumissil Microsystems" (id 6) (at 59.055 219.71 0)
+      (effects (font (size 1.27 1.27)) hide)
+    )
+    (property "Mfg Part #" "IS31FL3743A-QULS4-TR" (id 7) (at 59.055 219.71 0)
+      (effects (font (size 1.27 1.27)) hide)
+    )
+    (property "Package/Footprint" "QFN-40" (id 8) (at 59.055 219.71 0)
       (effects (font (size 1.27 1.27)) hide)
     )
@@
       (effects (font (size 1.27 1.27)) hide)
     )
-    (property "Datasheet" "http://ww1.microchip.com/downloads/en/DeviceDoc/20001952C.pdf" (id 3) (at 148.59 219.71 0)
-      (effects (font (size 1.27 1.27)) hide)
-    )
-    (property "Description / Value" "10MHz 16 POR SPI SOIC-28_300mil  I/O Expanders ROHS" (id 4) (at 148.59 219.71 0)
-      (effects (font (size 1.27 1.27)) hide)
-    )
-    (property "LCSC" "C47023" (id 5) (at 148.59 219.71 0)
-      (effects (font (size 1.27 1.27)) hide)
-    )
-    (property "Manufacturer" "Microchip Tech" (id 6) (at 148.59 219.71 0)
-      (effects (font (size 1.27 1.27)) hide)
-    )
-    (property "Mfg Part #" "MCP23S17T-E/SO" (id 7) (at 148.59 219.71 0)
-      (effects (font (size 1.27 1.27)) hide)
-    )
-    (property "Package/Footprint" "SOIC-28_7.5x17.9x1.27P" (id 8) (at 148.59 219.71 0)
+    (property "Datasheet" "https://datasheet.lcsc.com/lcsc/2106070633_Lumissil-Microsystems-IS31FL3743A-QULS4-TR_C2678953.pdf" (id 3) (at 148.59 219.71 0)
+      (effects (font (size 1.27 1.27)) hide)
+    )
+    (property "Description / Value" "UQFN-40(5x5)  LED Drivers ROHS" (id 4) (at 148.59 219.71 0)
+      (effects (font (size 1.27 1.27)) hide)
+    )
+    (property "LCSC" "C2678953" (id 5) (at 148.59 219.71 0)
+      (effects (font (size 1.27 1.27)) hide)
+    )
+    (property "Manufacturer" "Lumissil Microsystems" (id 6) (at 148.59 219.71 0)
+      (effects (font (size 1.27 1.27)) hide)
+    )
+    (property "Mfg Part #" "IS31FL3743A-QULS4-TR" (id 7) (at 148.59 219.71 0)
+      (effects (font (size 1.27 1.27)) hide)
+    )
+    (property "Package/Footprint" "QFN-40" (id 8) (at 148.59 219.71 0)
       (effects (font (size 1.27 1.27)) hide)
     )
@@
     (pin "2")
   )
-  (symbol (lib_id "vakeyboard:R") (at 57.785 244.475 270) (unit 1)
+  (symbol (lib_id "vakeyboard:R 10 kOhm") (at 57.785 244.475 270) (unit 1)
     (in_bom yes) (on_board yes) (fields_autoplaced)
     (property "Reference" "R2" (id 0) (at 57.785 241.3 90))
-    (property "Value" "R" (id 1) (at 57.785 244.475 90)
-      (effects (font (size 1.27 1.27)) hide)
-    )
-    (property "Footprint" "Footprints:R_0402_1005Metric" (id 2) (at 57.785 242.697 90)
-      (effects (font (size 1.27 1.27)) hide)
-    )
-    (property "Datasheet" "https://datasheet.lcsc.com/lcsc/2206010100_UNI-ROYAL-Uniroyal-Elec-0402WGF1002TCE_C25744.pdf" (id 3) (at 57.785 244.475 0)
-      (effects (font (size 1.27 1.27)) hide)
-    )
-    (property "Description / Value" "1/16W Thick Film Resistors 50V ±1% ±100ppm/℃ -55℃~+155℃ 10kΩ 0402  Chip Resistor - Surface Mount ROHS" (id 4) (at 57.785 244.475 0)
-      (effects (font (size 1.27 1.27)) hide)
-    )
-    (property "LCSC" "C25744" (id 5) (at 57.785 244.475 0)
-      (effects (font (size 1.27 1.27)) hide)
-    )
-    (property "Manufacturer" "UNI-ROYAL(Uniroyal Elec)" (id 6) (at 57.785 244.475 0)
-      (effects (font (size 1.27 1.27)) hide)
-    )
-    (property "Mfg Part #" "0402WGF1002TCE" (id 7) (at 57.785 244.475 0)
-      (effects (font (size 1.27 1.27)) hide)
-    )
-    (property "Package/Footprint" "0402" (id 8) (at 57.785 244.475 0)
-      (effects (font (size 1.27 1.27)) hide)
-    )
-    (property "Type" "SMD" (id 9) (at 57.785 244.475 0)
+    (property "Value" "R 10 kOhm" (id 1) (at 57.785 244.475 90)
+      (effects (font (size 1.27 1.27)) hide)
+    )
+    (property "Footprint" "Footprints:R_0402_1005Metric" (id 2) (at 23.495 243.205 0)
+      (effects (font (size 1.27 1.27)) hide)
+    )
+    (property "Datasheet" "https://datasheet.lcsc.com/lcsc/2206010100_UNI-ROYAL-Uniroyal-Elec-0402WGF1002TCE_C25744.pdf" (id 3) (at 41.275 245.745 0)
+      (effects (font (size 1.27 1.27)) hide)
+    )
+    (property "Description / Value" "1/16W Thick Film Resistors 50V ±1% ±100ppm/℃ -55℃~+155℃ 10kΩ 0402  Chip Resistor - Surface Mount ROHS" (id 4) (at 33.655 245.745 0)
+      (effects (font (size 1.27 1.27)) hide)
+    )
+    (property "LCSC" "C25744" (id 5) (at 31.115 244.475 0)
+      (effects (font (size 1.27 1.27)) hide)
+    )
+    (property "Manufacturer" "UNI-ROYAL(Uniroyal Elec)" (id 6) (at 38.735 245.745 0)
+      (effects (font (size 1.27 1.27)) hide)
+    )
+    (property "Mfg Part #" "0402WGF1002TCE" (id 7) (at 36.195 245.745 0)
+      (effects (font (size 1.27 1.27)) hide)
+    )
+    (property "Package/Footprint" "0402" (id 8) (at 28.575 244.475 0)
+      (effects (font (size 1.27 1.27)) hide)
+    )
+    (property "Type" "SMD" (id 9) (at 26.035 244.475 0)
       (effects (font (size 1.27 1.27)) hide)
     )
@@
     )
     (path "/ca65d83e-aa54-4c6c-bf1f-5c5c70a2d0ea"
-      (reference "R2") (unit 1) (value "R") (footprint "Footprints:R_0402_1005Metric")
+      (reference "R2") (unit 1) (value "R 10 kOhm") (footprint "Footprints:R_0402_1005Metric")
     )
     (path "/3339839e-4b3c-4af7-b282-24992a29ad74"
-      (reference "R3") (unit 1) (value "R") (footprint "Footprints:R_0402_1005Metric")
+      (reference "R3") (unit 1) (value "R 10 kOhm") (footprint "Footprints:R_0402_1005Metric")
     )
     (path "/6b4cfe13-64f5-4676-92bf-90e70977ec13"
